File: hardware/pcb/stm32-environmental-control-system/stm32-environmental-control-system.kicad_pcb (KiCad board)
At the start: 2 copper layers, 102.8 x 108.5 mm, 11 parts, among them J1 POWER, J10 FAN_POWER_IN, J2 DIGITAL_10, J3 ANALOG, J4 DIGITAL_8, J5 TEMP_SENSOR, J6 OLED, J7 MOSFET_CTRL, J8 FAN, J9 MOSFET_POWER

Commit message: cretaed gerbers pcb ready to order
Parts:
- moved RV1 12.7 mm to (89.8, 142.0)
- moved J7 12.2 mm to (133.0, 145.5)
- moved J5 10.8 mm to (90.5, 87.9)
- moved J6 8.40 mm to (144.7, 78.7)
Routing:
- net /GND: track 441.1 -> 395.9 mm
- net /3V3: track 177.7 -> 144.4 mm
- net /A1_PA1: track 65.8 -> 52.3 mm
- net /A0_PA0: track 46.3 -> 35.5 mm
- net /D14_PB9_SDA: track 24.9 -> 16.4 mm
- net /D15_PB8_SCL: track 21.3 -> 13.1 mm
- net /A2_PA4: track 46.9 -> 44.3 mm
Other:
- board size 102.8 x 108.5 mm -> 80.7 x 93.8 mm
